File: IrisV1/Sensors.kicad_sch (KiCad schematic)
At the start: 8 parts, among them U1 LSM6DSV80XTR, U18 MS561101BA03-50, U20 BMI323

Commit message: Symbol changes to use common library in Iris
Parts:
- A3: footprint Baro 1:XDCR_LPS22DFTR -> UNSW Rocketry Library:XDCR_LPS22DFTR; symbol Barometer:LPS22DFTR -> UNSW Rocketry library:LPS22DFTR
- U1: footprint Acc 1:QFN_LSM6DSV80XTR_STM -> UNSW Rocketry Library:QFN_LSM6DSV80XTR_STM; symbol IMU:LSM6DSV80XTR -> UNSW Rocketry library:LSM6DSV80XTR
- U18: footprint ms5611:SON8_MS5611_TEC -> UNSW Rocketry Library:SON8_MS5611_TEC; symbol high-alt Baro:MS561101BA03-50 -> UNSW Rocketry library:MS561101BA03-50
- U20: footprint BMI323:BMI323_BOS -> UNSW Rocketry Library:BMI323_BOS; symbol 16g acc:BMI323 -> UNSW Rocketry library:BMI323
Changed lines of the file:
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@@
 	)
 	(symbol
-		(lib_id "Barometer:LPS22DFTR")
+		(lib_id "UNSW Rocketry library:LPS22DFTR")
 		(at 237.49 41.91 0)
 		(mirror y)
@@
 			)
 		)
-		(property "Footprint" "Baro 1:XDCR_LPS22DFTR"
+		(property "Footprint" "UNSW Rocketry Library:XDCR_LPS22DFTR"
 			(at 237.49 41.91 0)
 			(hide yes)
@@
 	)
 	(symbol
-		(lib_id "16g acc:BMI323")
+		(lib_id "UNSW Rocketry library:BMI323")
 		(at 212.09 71.12 0)
 		(unit 1)
@@
 			)
 		)
-		(property "Footprint" "BMI323:BMI323_BOS"
+		(property "Footprint" "UNSW Rocketry Library:BMI323_BOS"
 			(at 212.09 71.12 0)
 			(hide yes)
@@
 	)
 	(symbol
-		(lib_id "IMU:LSM6DSV80XTR")
+		(lib_id "UNSW Rocketry library:LSM6DSV80XTR")
 		(at 121.92 67.31 0)
 		(unit 1)
@@
 			)
 		)
-		(property "Footprint" "Acc 1:QFN_LSM6DSV80XTR_STM"
-			(at 121.92 67.31 0)
+		(property "Footprint" "UNSW Rocketry Library:QFN_LSM6DSV80XTR_STM"
+			(at 122.682 55.372 0)
 			(hide yes)
 			(show_name no)
@@
 		)
 		(property "Datasheet" "https://www.st.com/resource/en/datasheet/lsm6dsv80x.pdf"
-			(at 121.92 67.31 0)
+			(at 121.412 51.308 0)
 			(hide yes)
 			(show_name no)
@@
 	)
 	(symbol
-		(lib_id "high-alt Baro:MS561101BA03-50")
+		(lib_id "UNSW Rocketry library:MS561101BA03-50")
 		(at 139.7 43.18 0)
 		(unit 1)
@@
 			)
 		)
-		(property "Footprint" "ms5611:SON8_MS5611_TEC"
+		(property "Footprint" "UNSW Rocketry Library:SON8_MS5611_TEC"
 			(at 139.7 43.18 0)
 			(hide yes)
