File: OneiroiV1/External.kicad_sch (KiCad schematic)
At the start: 24 parts, among them J10 MSD-10-C, J12 Conn_01x06, J3 USB4110GFA, J9 MSD-10-C, U16 ESDS302DBVR, U17 ESDS302DBVR, U24 ESDS302DBVR, U25 ESDS302DBVR

Commit message: Oneiroi Changes
All 3D models and footprints updated to common library, silkscreening must be re-done.
Parts:
- J10, J9: footprint locking microSD:CUI_MSD-10-C -> UNSW Rocketry Library:CUI_MSD-10-C; symbol locking microSD:MSD-10-C -> UNSW Rocketry Library:MSD-10-C
- J3: footprint USB:GCT_USB4110GFA -> UNSW Rocketry Library:GCT_USB4110GFA; symbol USB Connector:USB4110GFA -> UNSW Rocketry Library:USB4110GFA
- U16, U17, U24, U25: footprint esd:DBV0005A_N -> UNSW Rocketry Library:DBV0005A_N; symbol 3V3 ESD:ESDS302DBVR -> UNSW Rocketry Library:ESDS302DBVR
Changed lines of the file:
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@@
 	)
 	(symbol
-		(lib_id "3V3 ESD:ESDS302DBVR")
+		(lib_id "UNSW Rocketry Library:ESDS302DBVR")
 		(at 233.68 157.48 0)
 		(unit 1)
@@
 			)
 		)
-		(property "Footprint" "esd:DBV0005A_N"
+		(property "Footprint" "UNSW Rocketry Library:DBV0005A_N"
 			(at 233.68 157.48 0)
 			(hide yes)
@@
 	)
 	(symbol
-		(lib_id "3V3 ESD:ESDS302DBVR")
+		(lib_id "UNSW Rocketry Library:ESDS302DBVR")
 		(at 238.76 82.55 0)
 		(unit 1)
@@
 			)
 		)
-		(property "Footprint" "esd:DBV0005A_N"
+		(property "Footprint" "UNSW Rocketry Library:DBV0005A_N"
 			(at 238.76 82.55 0)
 			(hide yes)
@@
 	)
 	(symbol
-		(lib_id "USB Connector:USB4110GFA")
+		(lib_id "UNSW Rocketry Library:USB4110GFA")
 		(at 144.78 58.42 0)
 		(unit 1)
@@
 			)
 		)
-		(property "Footprint" "USB:GCT_USB4110GFA"
+		(property "Footprint" "UNSW Rocketry Library:GCT_USB4110GFA"
 			(at 144.78 58.42 0)
 			(hide yes)
@@
 	)
 	(symbol
-		(lib_id "locking microSD:MSD-10-C")
+		(lib_id "UNSW Rocketry Library:MSD-10-C")
 		(at 68.58 138.43 0)
 		(unit 1)
@@
 			)
 		)
-		(property "Footprint" "locking microSD:CUI_MSD-10-C"
+		(property "Footprint" "UNSW Rocketry Library:CUI_MSD-10-C"
 			(at 68.58 138.43 0)
 			(hide yes)
@@
 	)
 	(symbol
-		(lib_id "locking microSD:MSD-10-C")
+		(lib_id "UNSW Rocketry Library:MSD-10-C")
 		(at 68.58 69.85 0)
 		(unit 1)
@@
 			)
 		)
-		(property "Footprint" "locking microSD:CUI_MSD-10-C"
+		(property "Footprint" "UNSW Rocketry Library:CUI_MSD-10-C"
 			(at 68.58 69.85 0)
 			(hide yes)
@@
 	)
 	(symbol
-		(lib_id "3V3 ESD:ESDS302DBVR")
+		(lib_id "UNSW Rocketry Library:ESDS302DBVR")
 		(at 214.63 39.37 0)
 		(unit 1)
@@
 			)
 		)
-		(property "Footprint" "esd:DBV0005A_N"
+		(property "Footprint" "UNSW Rocketry Library:DBV0005A_N"
 			(at 214.63 39.37 0)
 			(hide yes)
@@
 	)
 	(symbol
-		(lib_id "3V3 ESD:ESDS302DBVR")
+		(lib_id "UNSW Rocketry Library:ESDS302DBVR")
 		(at 233.68 138.43 0)
 		(unit 1)
@@
 			)
 		)
-		(property "Footprint" "esd:DBV0005A_N"
+		(property "Footprint" "UNSW Rocketry Library:DBV0005A_N"
 			(at 233.68 138.43 0)
 			(hide yes)
