File: OneiroiV1/OneroiV1.kicad_sch (KiCad schematic)
At the start: 23 parts, among them J7 Conn_02x02_Odd_Even, U3 ESP32-S3-WROOM-1U-N4, U5 CVJ10F30_LF

Commit message: Oneiroi Changes
All 3D models and footprints updated to common library, silkscreening must be re-done.
Parts:
- LS1: footprint low volt buzzer:SPKR_CMI-1295-03TH -> UNSW Rocketry Library:SPKR_CMI-1295-03TH; symbol low volt buzzer:CMI-1295-03TH -> UNSW Rocketry Library:CMI-1295-03TH
- LS2: footprint better buzzer:CUI_CPI-1375-80T -> UNSW Rocketry Library:CUI_CPI-1375-80T; symbol better buzzer:CPI-1375-80T -> UNSW Rocketry Library:CPI-1375-80T
- U3: footprint ESP32-S3:XCVR_ESP32-S3-WROOM-1U-N4 -> UNSW Rocketry Library:XCVR_ESP32-S3-WROOM-1U-N4; symbol ESP32-S3:ESP32-S3-WROOM-1U-N4 -> UNSW Rocketry Library:ESP32-S3-WROOM-1U-N4
- U5: footprint Diode Chip:UFV_TOS -> UNSW Rocketry Library:UFV_TOS; symbol Double Diode:CVJ10F30_LF -> UNSW Rocketry Library:CVJ10F30_LF
Changed lines of the file:
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@@
 	)
 	(junction
-		(at 254 40.64)
-		(diameter 0)
-		(color 0 0 0 0)
-	)
-	(junction
 		(at 128.27 102.87)
 		(diameter 0)
@@
 	)
 	(junction
+		(at 254 40.64)
+		(diameter 0)
+		(color 0 0 0 0)
+	)
+	(junction
 		(at 245.11 53.34)
 		(diameter 0)
@@
 	)
 	(junction
-		(at 128.27 113.03)
+		(at 254 50.8)
 		(diameter 0)
 		(color 0 0 0 0)
 	)
 	(junction
-		(at 254 50.8)
+		(at 128.27 113.03)
 		(diameter 0)
 		(color 0 0 0 0)
@@
 	(wire
 		(pts
+			(xy 254 50.8) (xy 274.32 50.8)
+		)
+		(stroke
+			(width 0)
+			(type default)
+		)
+	)
+	(wire
+		(pts
 			(xy 116.84 162.56) (xy 119.38 162.56)
 		)
@@
 	(wire
 		(pts
+			(xy 254 40.64) (xy 274.32 40.64)
+		)
+		(stroke
+			(width 0)
+			(type default)
+		)
+	)
+	(wire
+		(pts
 			(xy 128.27 62.23) (xy 132.08 62.23)
 		)
@@
 	(wire
 		(pts
-			(xy 254 50.8) (xy 248.92 50.8)
+			(xy 248.92 50.8) (xy 254 50.8)
 		)
 		(stroke
@@
 	(wire
 		(pts
-			(xy 254 40.64) (xy 274.32 40.64)
-		)
-		(stroke
-			(width 0)
-			(type default)
-		)
-	)
-	(wire
-		(pts
 			(xy 158.75 163.83) (xy 163.83 163.83)
 		)
@@
 	(wire
 		(pts
-			(xy 254 50.8) (xy 274.32 50.8)
-		)
-		(stroke
-			(width 0)
-			(type default)
-		)
-	)
-	(wire
-		(pts
 			(xy 96.52 46.99) (xy 97.79 46.99)
 		)
@@
 	(wire
 		(pts
-			(xy 254 40.64) (xy 245.11 40.64)
+			(xy 245.11 40.64) (xy 254 40.64)
 		)
 		(stroke
@@
 	)
 	(symbol
-		(lib_id "ESP32-S3:ESP32-S3-WROOM-1U-N4")
+		(lib_id "UNSW Rocketry Library:ESP32-S3-WROOM-1U-N4")
 		(at 113.03 67.31 0)
 		(unit 1)
@@
 			)
 		)
-		(property "Footprint" "ESP32-S3:XCVR_ESP32-S3-WROOM-1U-N4"
+		(property "Footprint" "UNSW Rocketry Library:XCVR_ESP32-S3-WROOM-1U-N4"
 			(at 113.03 67.31 0)
 			(hide yes)
@@
 	)
 	(symbol
-		(lib_id "Double Diode:CVJ10F30_LF")
+		(lib_id "UNSW Rocketry Library:CVJ10F30_LF")
 		(at 218.44 66.04 0)
 		(unit 1)
@@
 			)
 		)
-		(property "Footprint" "Diode Chip:UFV_TOS"
+		(property "Footprint" "UNSW Rocketry Library:UFV_TOS"
 			(at 243.84 62.992 0)
 			(hide yes)
@@
 	)
 	(symbol
-		(lib_id "low volt buzzer:CMI-1295-03TH")
+		(lib_id "UNSW Rocketry Library:CMI-1295-03TH")
 		(at 276.86 45.72 0)
 		(unit 1)
@@
 			)
 		)
-		(property "Footprint" "low volt buzzer:SPKR_CMI-1295-03TH"
+		(property "Footprint" "UNSW Rocketry Library:SPKR_CMI-1295-03TH"
 			(at 276.86 45.72 0)
 			(hide yes)
@@
 	)
 	(symbol
-		(lib_id "better buzzer:CPI-1375-80T")
+		(lib_id "UNSW Rocketry Library:CPI-1375-80T")
 		(at 254 45.72 0)
 		(unit 1)
@@
 			)
 		)
-		(property "Footprint" "better buzzer:CUI_CPI-1375-80T"
+		(property "Footprint" "UNSW Rocketry Library:CUI_CPI-1375-80T"
 			(at 254 45.72 0)
 			(hide yes)
